Commit message: add base frame

File: config/gazebo_ur5_with_robotiq_2f_85.urdf (robot description, URDF)
Before this commit: robot ur5_with_robotiq_2f_85, 21 links, 20 joints
Links:
- removed link world
- added link frame, mass 40.0; collision mesh filename=package://ur5_gripper_moveit/meshes/frame/collision/frame.s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; visual mesh filename=package://ur5_gripper_moveit/meshes/frame/visual/frame.dae
Joints:
- joint virtual_base: origin xyz=0 0 0 rpy=0 0 0 -> xyz=0 0 0.87 rpy=0 0 1.57; parent world -> frame

Commit message: update frame in real robot control

File: config/gazebo_ur5_with_robotiq_2f_85.urdf (robot description, URDF)
Before this commit: robot ur5_with_robotiq_2f_85, 21 links, 20 joints
Links:
- added link world
Joints:
- added joint frame_base: type fixed, parent frame, child base_link, origin xyz=0 0 0.87 rpy=0 0 1.57
- joint virtual_base: child base_link -> frame; origin xyz=0 0 0.87 rpy=0 0 1.57 -> xyz=0 0 0 rpy=0 0 0; parent frame -> world

Commit message: add scanner to the scene

File: config/gazebo_ur5_with_robotiq_2f_85.urdf (robot description, URDF)
Before this commit: robot ur5_with_robotiq_2f_85, 22 links, 21 joints
Links:
- added link scanner, mass 40.0; collision mesh filename=package://ur5_gripper_moveit/meshes/scanner/collision/scann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; visual mesh filename=package://ur5_gripper_moveit/meshes/scanner/visual/scanner.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
Joints:
- added joint scanner_frame: type fixed, parent frame, child scanner, origin xyz=0 1.53 1.681 rpy=-1.57 0 3.14

Commit message: realsense with bug

File: config/gazebo_ur5_with_robotiq_2f_85.urdf (robot description, URDF)
Before this commit: robot ur5_with_robotiq_2f_85, 23 links, 22 joints
Links:
- added link realsense, mass 40.0; collision mesh filename=package://ur5_gripper_moveit/meshes/realsense/collision/rea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; visual mesh filename=package://ur5_gripper_moveit/meshes/realsense/visual/realse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
Joints:
- added joint tool_realsense: type fixed, parent tool0, child realsense, origin xyz=0 0 0 rpy=0 0 0

Commit message: fixed wrong origins

File: config/gazebo_ur5_with_robotiq_2f_85.urdf (robot description, URDF)
Before this commit: robot ur5_with_robotiq_2f_85, 24 links, 23 joints
Links:
- link realsense: mass 40.0 -> 0.4
Joints:
- joint frame_base: origin xyz=0 0 0.87 rpy=0 0 1.57 -> xyz=0 0 0 rpy=0 0 1.57
- joint scanner_frame: origin xyz=0 1.53 1.681 rpy=-1.57 0 3.14 -> xyz=-0.025 0.67 0.817 rpy=-1.57 0 3.14
- joint tool_realsense: origin xyz=0 0 0 rpy=0 0 0 -> xyz=0 0 0 rpy=1.57 0 -1.57 
- joint virtual_base: origin xyz=0 0 0 rpy=0 0 0 -> xyz=0 0 0.857 rpy=0 0 0

Commit message: correct robotiq position

File: config/gazebo_ur5_with_robotiq_2f_85.urdf (robot description, URDF)
Before this commit: robot ur5_with_robotiq_2f_85, 24 links, 23 joints
Joints:
- joint frame_base: origin xyz=0 0 0 rpy=0 0 1.57 -> xyz=0 0 0.01 rpy=0 0 1.57
- joint robotiq_85_base_joint: origin xyz=0 0 0.004 rpy=0 -1.5707963267948966 3.141592653589793 -> xyz=0 0 0.004 rpy=0 -1.5707963267948966 1.5707963267948966
- joint scanner_frame: origin xyz=-0.025 0.67 0.817 rpy=-1.57 0 3.14 -> xyz=-0.025 0.66 0.775 rpy=-1.57 0 3.14
- joint tool_realsense: origin xyz=0 0 0 rpy=1.57 0 -1.57  -> xyz=0 0 0 rpy=1.57 0 3.14 

Commit message: use correct frame model

File: config/gazebo_ur5_with_robotiq_2f_85.urdf (robot description, URDF)
Before this commit: robot ur5_with_robotiq_2f_85, 24 links, 23 joints
Joints:
- joint scanner_frame: origin xyz=-0.025 0.66 0.775 rpy=-1.57 0 3.14 -> xyz=-0.015 0.67 0.775 rpy=-1.57 0 3.14

Commit message: add tray

File: config/gazebo_ur5_with_robotiq_2f_85.urdf (robot description, URDF)
Before this commit: robot ur5_with_robotiq_2f_85, 24 links, 23 joints
Links:
- added link tray, mass 40.0; collision mesh filename=package://ur5_gripper_moveit/meshes/tray/collision/grasping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; visual mesh filename=package://ur5_gripper_moveit/meshes/tray/visual/grasping_tr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
Joints:
- added joint frame_tray: type fixed, parent frame, child tray, origin xyz=0.015 0.54 0 rpy=0 0 1.57 
